Commit message: added meshes to urdf

File: urdf/p626.urdf (robot description, URDF)
Before this commit: robot Project_626, 3 links, 2 joints
Links:
- link base_link: geometry visual mesh filename=file:///home/coppo/urdf_ws/src/nav_launch/meshes/p626.dae scale=0.01 0.01 0.01
- link laser_link: geometry 
